Commit message: 部分运动学代码

File: src/robot_description/urdf/xarm6/xarm6.urdf.xacro (robot description, xacro)
@@ -122,17 +122,3 @@
     <limit lower="-3.14" upper="3.14" effort="20.0" velocity="3.14"/>
   </joint>
-  <!-- 末端执行器 - 明显标记 -->
-  <link name="flange">
-    <visual>
-      <geometry>
-        <sphere radius="0.03"/>
-      </geometry>
-      <material name="red"/>
-    </visual>
-  </link>
-  <joint name="flange_joint" type="fixed">
-    <parent link="link6"/>
-    <child link="flange"/>
-    <origin xyz="0.15 0 0" rpy="0 0 0"/>
-  </joint>
 </robot>
